File: PCB/Cmote/Cmote.kicad_pcb (KiCad board)
At the start: 4 copper layers, 21.2 x 29.9 mm, 20 parts, among them J1 TSOP 1738, J2 UPDI_Pad, J3 Power_Pad, J5 DevPad1, J6 DevPad2, Q1 Si2302CDS-T1-GE3, U1 ATTINY1616-MNR, U2 IR16-213C/L510/TR8, U3 CH340N_C2977777

Commit message: silkscreen "art"
Parts:
- renumbered C_v3_USB0 to C5
Other:
- board text added: "3"
- board text added: ":"
- board text added: "Cmote v1.0"
- board text added: "mrow"
