File: PCB/Cmote/Cmote.kicad_pcb (KiCad board)
At the start: 4 copper layers, 21.2 x 29.9 mm, 20 parts, among them J1 TSOP 1738, J2 UPDI_Pad, J3 Power_Pad, J5 DevPad1, J6 DevPad2, Q1 Si2302CDS-T1-GE3, U1 ATTINY1616-MNR, U2 IR16-213C/L510/TR8, U3 CH340N_C2977777

Commit message: update via to prevent solder wicking
Routing:
- net GND: vias 11 -> 7
Changed lines of the file:
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@@
 	)
 	(via
-		(at 148.765 110.0372)
-		(size 0.6)
-		(drill 0.3)
-		(layers "F.Cu" "B.Cu")
-		(net 2)
-	)
-	(via
-		(at 149.765 109.0372)
-		(size 0.6)
-		(drill 0.3)
-		(layers "F.Cu" "B.Cu")
-		(net 2)
-	)
-	(via
-		(at 148.765 109.0372)
-		(size 0.6)
-		(drill 0.3)
-		(layers "F.Cu" "B.Cu")
-		(net 2)
-	)
-	(via
-		(at 149.765 110.0372)
+		(at 149.265 109.5372)
 		(size 0.6)
 		(drill 0.3)
@@
 		(size 0.6)
 		(drill 0.3)
-		(layers "F.Cu" "B.Cu")
-		(net 2)
-	)
-	(via
-		(at 149.265 109.5372)
-		(size 0.6)
-		(drill 0.3)
