File: PCB/Cmote/Cmote.kicad_sch (KiCad schematic)
At the start: 17 parts, among them J1 TSOP 1738, J2 UPDI_Pad, J3 Power_Pad, J5 DevPad1, J6 DevPad2, Q1 Si2302CDS-T1-GE3, U1 ATTINY1616-MNR, U2 IR16-213C/L510/TR8, U3 CH340N_C2977777

Commit message: pcb done
Parts:
- added R3, R4: 5.1k, easyeda2kicad:R0402, symbol Device:R_Small
- added USB1: HYCW671-USBC14-115B, easyeda2kicad:USB-SMD_HYCW671-USBC14-115B, symbol easyeda2kicad:HYCW671-USBC14-115B
- J5, J6: now left out of the parts list
- renumbered C_VCC_USB2 to C1, C_VCC_USB1 to C2, C_IR_RX0 to C3, C_MCU0 to C4
Connections:
- net +5V: now also J2.2 (Pin_2), J3.1 (Pin_1), USB1.A4 (VBUS), USB1.A9 (VBUS), USB1.B4 (VBUS), USB1.B9 (VBUS); no longer J2.VDD (Pin_2), J3.Vcc (Pin_1)
- net GND: now also J2.3 (Pin_3), J3.2 (Pin_2), R3.1, R4.2, USB1.1 (GND), USB1.2 (GND), USB1.3 (GND), USB1.4 (GND), USB1.A1 (GND), USB1.A12 (GND), USB1.B1 (GND), USB1.B12 (GND); no longer J2.GND (Pin_3), J3.GND (Pin_2)
- net USB_D+: now also USB1.A6 (DP1), USB1.B6 (DP2)
- net USB_D-: now also USB1.A7 (DN1), USB1.B7 (DN2)
- net at R_UPDI0.2: now also J2.1 (Pin_1); no longer J2.UPDI (Pin_1)
- new net: R3.2, USB1.B5 (CC2)
- new net: R4.1, USB1.A5 (CC1)
Other:
- note added: "USB-C Plug"

Commit message: silkscreen "art"
Parts:
- renumbered C_v3_USB0 to C5
Changed lines of the file:
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@@
 		(on_board yes)
 		(dnp no)
-		(property "Reference" "C_v3_USB0"
-			(at 83.058 82.55 90)
+		(property "Reference" "C5"
+			(at 80.518 82.296 90)
 			(effects
 				(font
@@
 			(project ""
 				(path "/463ee1d0-3616-4553-a2de-372769077643"
-					(reference "C_v3_USB0")
+					(reference "C5")
 					(unit 1)
 				)

Commit message: updated parts to get more basic assembly
Parts:
- C1: LCSC Part C527010 -> C19666; MPN CC0402KRX5R7BB474 -> CL10A475KO8NNNC; Manufacturer YAGEO -> Samsung Electro-Mechanics
- C2, C3, C4, C5: LCSC Part C106204 -> C1525; MPN CC0402KRX5R7BB104 -> CL05B104KO5NNNC; Manufacturer YAGEO -> Samsung Electro-Mechanics
- R2: LCSC Part C106232 -> C25076; MPN RC0402FR-07100RL -> 0402WGF1000TCE; Manufacturer YAGEO -> UNI-ROYAL(Uniroyal Elec)
- R3, R4: LCSC Part C105872 -> C25905; MPN RC0402FR-075K1L -> 0402WGF5101TCE; Manufacturer YAGEO -> UNI-ROYAL(Uniroyal Elec)
- R_UPDI0: LCSC Part C114877 -> C25117; MPN RC0402FR-07470RL -> 0402WGF4700TCE; Manufacturer YAGEO -> UNI-ROYAL(Uniroyal Elec)
